File: pcb/MAD.kicad_pcb (KiCad board)
At the start: 2 copper layers, 36 x 47 mm, 48 parts, among them J1 Conn_01x06_Pin, J2 Conn_01x06_Socket, Q1 AO3416A, Q10 AO3419A, Q11 AO3416A, Q12 AO3416A, Q2 AO3419A, Q3 AO3416A, Q4 AO3419A, Q5 AO3416A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

Commit message: Optimize resistor values
Parts:
- R2, R3, R4, R5, R6, R7, R8: value 22 -> 0R1
Changed lines of the file:
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@@
         (effects (font (size 1 1) (thickness 0.15)))
     )
-    (fp_text value "22" (at 0 -1.905 90) (layer "F.Fab")
+    (fp_text value "0R1" (at 0 -1.905 90) (layer "F.Fab")
         (effects (font (size 1 1) (thickness 0.15)))
     )
@@
         (effects (font (size 1 1) (thickness 0.15)))
     )
-    (fp_text value "22" (at 0 1.82 90) (layer "F.Fab")
+    (fp_text value "0R1" (at 0 1.82 90) (layer "F.Fab")
         (effects (font (size 1 1) (thickness 0.15)))
     )
@@
         (effects (font (size 1 1) (thickness 0.15)))
     )
-    (fp_text value "22" (at 0 -2.032 90) (layer "F.Fab")
+    (fp_text value "0R1" (at 0 -2.032 90) (layer "F.Fab")
         (effects (font (size 1 1) (thickness 0.15)))
     )
@@
         (effects (font (size 1 1) (thickness 0.15)))
     )
-    (fp_text value "22" (at 0 1.82 90) (layer "F.Fab")
+    (fp_text value "0R1" (at 0 1.82 90) (layer "F.Fab")
         (effects (font (size 1 1) (thickness 0.15)))
     )
@@
         (effects (font (size 1 1) (thickness 0.15)))
     )
-    (fp_text value "22" (at 0 -2.032 90) (layer "F.Fab")
+    (fp_text value "0R1" (at 0 -2.032 90) (layer "F.Fab")
         (effects (font (size 1 1) (thickness 0.15)))
     )
@@
         (effects (font (size 1 1) (thickness 0.15)))
     )
-    (fp_text value "22" (at 0 -2.032 90) (layer "F.Fab")
+    (fp_text value "0R1" (at 0 -2.032 90) (layer "F.Fab")
         (effects (font (size 1 1) (thickness 0.15)))
     )
@@
         (effects (font (size 1 1) (thickness 0.15)))
     )
-    (fp_text value "22" (at 0 1.82 90) (layer "F.Fab")
+    (fp_text value "0R1" (at 0 1.82 90) (layer "F.Fab")
         (effects (font (size 1 1) (thickness 0.15)))
     )
