File: pcb/MAD.kicad_pcb (KiCad board)
At the start: 2 copper layers, 36 x 47 mm, 48 parts, among them J1 Conn_01x06_Pin, J2 Conn_01x06_Socket, Q1 AO3416A, Q10 AO3419A, Q11 AO3416A, Q12 AO3416A, Q2 AO3419A, Q3 AO3416A, Q4 AO3419A, Q5 AO3416A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

Commit message: Change SPI-Bus names
Connections:
- net /MISO renamed /SO
- net /MOSI renamed /SI

Commit message: Add ATtiny __06 to design
Parts:
- U1: value ATtiny406-S -> ATtiny__06-S
Changed lines of the file:
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@@
     (property "Sheetname" "")
     (property "Vendor" "HTL")
-    (property "VendorId" "103335")
+    (property "VendorId" "103335,103450")
     (property "ki_description" "20MHz, 4kB Flash, 256B SRAM, 128B EEPROM, SOIC-20")
     (property "ki_keywords" "AVR 8bit Microcontroller tinyAVR")
@@
         (effects (font (size 1 1) (thickness 0.15)))
     )
-    (fp_text value "ATtiny406-S" (at 0 7.35 90) (layer "F.Fab")
+    (fp_text value "ATtiny__06-S" (at 0 7.35 90) (layer "F.Fab")
         (effects (font (size 1 1) (thickness 0.15)))
     )

Commit message: Optimize current consumption
Parts:
- R2, R3, R4, R5, R6, R7, R8: value 0R1 -> 15
Changed lines of the file:
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@@
     (property "Sheetname" "")
     (property "Vendor" "HTL")
-    (property "VendorId" "102901")
+    (property "VendorId" "102916")
     (property "ki_description" "Resistor")
     (property "ki_keywords" "R res resistor")
@@
         (effects (font (size 1 1) (thickness 0.15)))
     )
-    (fp_text value "0R1" (at 0 -1.905 90) (layer "F.Fab")
+    (fp_text value "15" (at 0 -1.905 90) (layer "F.Fab")
         (effects (font (size 1 1) (thickness 0.15)))
     )
@@
     (property "Sheetname" "")
     (property "Vendor" "HTL")
-    (property "VendorId" "102901")
+    (property "VendorId" "102916")
     (property "ki_description" "Resistor")
     (property "ki_keywords" "R res resistor")
@@
         (effects (font (size 1 1) (thickness 0.15)))
     )
-    (fp_text value "0R1" (at 0 1.82 90) (layer "F.Fab")
+    (fp_text value "15" (at 0 1.82 90) (layer "F.Fab")
         (effects (font (size 1 1) (thickness 0.15)))
     )
@@
     (property "Sheetname" "")
     (property "Vendor" "HTL")
-    (property "VendorId" "102901")
+    (property "VendorId" "102916")
     (property "ki_description" "Resistor")
     (property "ki_keywords" "R res resistor")
@@
         (effects (font (size 1 1) (thickness 0.15)))
     )
-    (fp_text value "0R1" (at 0 -2.032 90) (layer "F.Fab")
+    (fp_text value "15" (at 0 -2.032 90) (layer "F.Fab")
         (effects (font (size 1 1) (thickness 0.15)))
     )
@@
     (property "Sheetname" "")
     (property "Vendor" "HTL")
-    (property "VendorId" "102901")
+    (property "VendorId" "102916")
     (property "ki_description" "Resistor")
     (property "ki_keywords" "R res resistor")
@@
         (effects (font (size 1 1) (thickness 0.15)))
     )
-    (fp_text value "0R1" (at 0 1.82 90) (layer "F.Fab")
+    (fp_text value "15" (at 0 1.82 90) (layer "F.Fab")
         (effects (font (size 1 1) (thickness 0.15)))
     )
@@
     (property "Sheetname" "")
     (property "Vendor" "HTL")
-    (property "VendorId" "102901")
+    (property "VendorId" "102916")
     (property "ki_description" "Resistor")
     (property "ki_keywords" "R res resistor")
@@
         (effects (font (size 1 1) (thickness 0.15)))
     )
-    (fp_text value "0R1" (at 0 -2.032 90) (layer "F.Fab")
+    (fp_text value "15" (at 0 -2.032 90) (layer "F.Fab")
         (effects (font (size 1 1) (thickness 0.15)))
     )
@@
     (property "Sheetname" "")
     (property "Vendor" "HTL")
-    (property "VendorId" "102901")
+    (property "VendorId" "102916")
     (property "ki_description" "Resistor")
     (property "ki_keywords" "R res resistor")
@@
         (effects (font (size 1 1) (thickness 0.15)))
     )
-    (fp_text value "0R1" (at 0 -2.032 90) (layer "F.Fab")
+    (fp_text value "15" (at 0 -2.032 90) (layer "F.Fab")
         (effects (font (size 1 1) (thickness 0.15)))
     )
@@
     (property "Sheetname" "")
     (property "Vendor" "HTL")
-    (property "VendorId" "102901")
+    (property "VendorId" "102916")
     (property "ki_description" "Resistor")
     (property "ki_keywords" "R res resistor")
@@
         (effects (font (size 1 1) (thickness 0.15)))
     )
-    (fp_text value "0R1" (at 0 1.82 90) (layer "F.Fab")
+    (fp_text value "15" (at 0 1.82 90) (layer "F.Fab")
         (effects (font (size 1 1) (thickness 0.15)))
     )
